File: eagle/gs.brd (EAGLE design)
At the start: 100.1 x 50 mm, 45 parts, among them J1 USB-B-MICRO, Q1 S8050, Q2 S8050, Q3 S8050, Q4 S8050, U1 LD1086DT33TR, U2 CP2102, U3 ESP32-SOLO-1, U4 E22-400M30S, X1 SMA

Commit message: Fixed ESP32-SOLO-1 used instead of ESP32-WROOM-32D
Parts:
- U3: value ESP32-SOLO-1 -> ESP32-WROOM-32D
Changed lines of the file:
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@@
 <attribute name="VALUE" x="20.701" y="2.921" size="1.27" layer="27"/>
 </element>
-<element name="U3" library="fossa" library_urn="urn:adsk.eagle:library:24422541" package="ESP32-SOLO-1" package3d_urn="urn:adsk.eagle:package:24422546/2" value="ESP32-SOLO-1" x="43.688" y="36.195" smashed="yes">
+<element name="U3" library="fossa" library_urn="urn:adsk.eagle:library:24422541" package="ESP32-SOLO-1" package3d_urn="urn:adsk.eagle:package:24422546/2" value="ESP32-WROOM-32D" x="43.688" y="36.195" smashed="yes">
 <attribute name="NAME" x="34.307" y="23.025" size="0.8128" layer="25" align="top-right"/>
-<attribute name="TME" value="ESP32-SOLO-1" x="94.488" y="22.225" size="1.778" layer="27" display="off"/>
+<attribute name="TME" value="ESP32-WROOM-32D" x="94.488" y="22.225" size="1.778" layer="27" display="off"/>
 </element>
 <element name="U4" library="fossa" library_urn="urn:adsk.eagle:library:24422541" package="E22-400M30S" package3d_urn="urn:adsk.eagle:package:24427036/2" value="E22-400M30S" x="75.692" y="19.812" smashed="yes" rot="R270">
