File: eagle/gs.sch (EAGLE design)
At the start: 45 parts, among them J1 USB-B-MICRO, Q1 S8050, Q2 S8050, Q3 S8050, Q4 S8050, U1 LD1086DT33TR, U2 CP2102, U3 ESP32-SOLO-1, U4 E22-400M30S, X1 SMA

Commit message: Fixed ESP32-SOLO-1 used instead of ESP32-WROOM-32D
Parts:
- U3: value ESP32-SOLO-1 -> ESP32-WROOM-32D; device fossa:ESP32-SOLO-1 -> fossa:ESP32-WROOM-32D
Changed lines of the file:
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@@
 </classes>
 <parts>
-<part name="U3" library="fossa" library_urn="urn:adsk.eagle:library:24422541" deviceset="ESP32-SOLO-1" device="" package3d_urn="urn:adsk.eagle:package:24422546/2"/>
+<part name="U3" library="fossa" library_urn="urn:adsk.eagle:library:24422541" deviceset="ESP32-WROOM-32D" device="" package3d_urn="urn:adsk.eagle:package:24422546/2"/>
 <part name="GND1" library="supply1" library_urn="urn:adsk.eagle:library:371" deviceset="GND" device=""/>
 <part name="GND2" library="supply1" library_urn="urn:adsk.eagle:library:371" deviceset="GND" device=""/>
